Commit message: :+1: update code for simulation

File: beaverbot_description/urdf/beaverbot.urdf.xacro (robot description, xacro)
@@ -20,9 +20,8 @@
     <collision>
       <geometry>
-        <box size="1.24 0.74 0.46"/>	<!-- rough robot size: x=1.24 y=0.74 z=0.46 -->
+        <box size="0.01 0.01 0.01"/>
       </geometry>
-      <origin rpy="0 0 0" xyz="0.395 0.0 0.12"/>
     </collision>
-    <!--<xacro:inertial_box mass="0.01" x="0.01" y="0.01" z="0.01" />-->
+    <xacro:inertial_box mass="0.01" x="0.01" y="0.01" z="0.01" />
   </link>
   <gazebo reference="base_link">
@@ -60,5 +59,5 @@
     <parent link="base_link"/>
     <child link="robot_center"/>
-    <origin xyz="0.415 0.0 0.0" />
+    <origin xyz="0 0.0 0.0" />
   </joint>
   <!-- ////////////////////////// Base Link and Wheel Connections and Links ////////////////////////// -->

File: beaverbot_description/urdf/properties.xacro (robot description, xacro)
@@ -19,5 +19,5 @@
   <xacro:property name="castor_plate_mass" value="0.12" />          <!-- updated -->
   <xacro:property name="castor_support_mass" value="0.1" />         <!-- updated -->
-  <xacro:property name="castor_mass" value="0.3" />                 <!-- updated -->
+  <xacro:property name="castor_mass" value="0.5" />                 <!-- updated -->
   <xacro:property name="top_support_mass" value="0.65" />           <!-- updated -->
   <xacro:property name="top_frame_yellow_mass" value="1.5" />       <!-- updated -->

Commit message: :+1: beaverbot: fix jumping problem

File: beaverbot_description/urdf/beaverbot.urdf.xacro (robot description, xacro)
@@ -69,5 +69,5 @@
   <xacro:default_zylinder_in_Y parent="base" child_name="wheel_support_left" mass="${wheel_support_mass}" length="0.13" radius="0.05" ox="-0.11" oy="0.155" oz="-0.061" roll="${pi/2}" yaw="0.0" pitch="0.0" color="Black" />
   <xacro:default_zylinder_in_Y parent="base" child_name="wheel_support_right" mass="${wheel_support_mass}" length="0.13" radius="0.05" ox="-0.11" oy="-0.155" oz="-0.061" roll="${pi/2}" yaw="0.0" pitch="0.0" color="Black" />
-  <xacro:default_zylinder_in_Z parent="top_support" child_name="lidar_base" mass="${lidar_base_mass}" length="0.025" radius="0.025" ox="0.01" oy="0.0" oz="0.015" roll="0.0" yaw="0.0" pitch="0.0" color="Black" />
+  <xacro:default_zylinder_in_Z parent="top_support" child_name="lidar_base" mass="${lidar_base_mass}" length="0.025" radius="0.025" ox="0.01" oy="0.0" oz="0.015" roll="0.0" yaw="0.0" pitch="0.0" color="Black"/>
   <!-- <xacro:default_zylinder_in_Z parent="front_frame_black" child_name="front_light_left" mass="${front_light_mass}" length="0.005" radius="0.025" ox="0.001" oy="0.175" oz="0.12" roll="0.0" pitch="${pi/2}" yaw="0.0" color="White" />
   <xacro:default_zylinder_in_Z parent="front_frame_black" child_name="front_light_right" mass="${front_light_mass}" length="0.005" radius="0.025" ox="0.001" oy="-0.175" oz="0.12" roll="0.0" pitch="${pi/2}" yaw="0.0" color="White" /> -->
@@ -78,6 +78,6 @@
   <!-- /////////////////////////////////////////////////////////////////////////////////////////////// -->
   <!-- ////////////////////////// Omnidirectional Wheels ////////////////////////// -->
-  <xacro:default_zylinder_in_Z parent="zylinder_base_support_left" child_name="zylinder_to_castor_left" mass="${zylinder_to_castor_mass}" length="0.35" radius="0.0175" ox="0.26" oy="0.0" oz="-0.04" yaw="0.0" pitch="0.0" roll="0.0" color="Black" />
-  <xacro:default_zylinder_in_Z parent="zylinder_base_support_right" child_name="zylinder_to_castor_right" mass="${zylinder_to_castor_mass}" length="0.35" radius="0.0175" ox="0.26" oy="0.0" oz="-0.04" yaw="0.0" pitch="0.0" roll="0.0" color="Black" />
+  <xacro:default_zylinder_in_Z parent="zylinder_base_support_left" child_name="zylinder_to_castor_left" mass="${zylinder_to_castor_mass}" length="0.35" radius="0.0175" ox="0.26" oy="0.0" oz="-0.04" yaw="0.0" pitch="0.0" roll="0.0" color="Black"/>
+  <xacro:default_zylinder_in_Z parent="zylinder_base_support_right" child_name="zylinder_to_castor_right" mass="${zylinder_to_castor_mass}" length="0.35" radius="0.0175" ox="0.26" oy="0.0" oz="-0.04" yaw="0.0" pitch="0.0" roll="0.0" color="Black"/>
   <xacro:default_box parent="zylinder_to_castor_left" child_name="castor_plate_left" mass="${castor_plate_mass}" sizex="0.07" sizey="0.10" sizez="0.005" ox="0.0" oy="0.0" oz="-0.175" yaw="0.0" pitch="0.0" roll="0.0" color="Black" />
   <xacro:default_box parent="zylinder_to_castor_right" child_name="castor_plate_right" mass="${castor_plate_mass}" sizex="0.07" sizey="0.10" sizez="0.005" ox="0.0" oy="0.0" oz="-0.175" yaw="0.0" pitch="0.0" roll="0.0" color="Black" />
@@ -86,8 +86,8 @@
   <xacro:default_box parent="castor_plate_right" child_name="castor_support_leftright" mass="${castor_support_mass}" sizex="0.03" sizey="0.005" sizez="0.09" ox="0.0" oy="0.0475" oz="-0.045" yaw="0.0" pitch="0.0" roll="0.0" color="Black" />
   <xacro:default_box parent="castor_plate_right" child_name="castor_support_rightright" mass="${castor_support_mass}" sizex="0.03" sizey="0.005" sizez="0.09" ox="0.0" oy="-0.0475" oz="-0.045" yaw="0.0" pitch="0.0" roll="0.0" color="Black" />
-  <xacro:default_zylinder_in_Y_with_collision parent="castor_plate_left" child_name="castor_leftleft" mass="${castor_mass}" length="0.045" radius="0.04" ox="0.0" oy="0.0225" oz="-0.075" roll="${pi/2}" yaw="0.0" pitch="0.0" color="Grey" />
-  <xacro:default_zylinder_in_Y_with_collision parent="castor_plate_left" child_name="castor_rightleft" mass="${castor_mass}" length="0.045" radius="0.04" ox="0.0" oy="-0.0225" oz="-0.075" roll="${pi/2}" yaw="0.0" pitch="0.0" color="Grey" />
-  <xacro:default_zylinder_in_Y_with_collision parent="castor_plate_right" child_name="castor_leftright" mass="${castor_mass}" length="0.045" radius="0.04" ox="0.0" oy="0.0225" oz="-0.075" roll="${pi/2}" yaw="0.0" pitch="0.0" color="Grey" />
-  <xacro:default_zylinder_in_Y_with_collision parent="castor_plate_right" child_name="castor_rightright" mass="${castor_mass}" length="0.045" radius="0.04" ox="0.0" oy="-0.0225" oz="-0.075" roll="${pi/2}" yaw="0.0" pitch="0.0" color="Grey" />
+  <xacro:default_zylinder_in_Y_with_collision parent="castor_plate_left" child_name="castor_leftleft" mass="${castor_mass}" length="0.045" radius="0.04" ox="0.0" oy="0.0225" oz="-0.075" roll="${pi/2}" yaw="0.0" pitch="0.0" color="Grey" mu1="${mu1}" mu2="${mu2}" kp="${kp}" kd="${kd}" />
+  <xacro:default_zylinder_in_Y_with_collision parent="castor_plate_left" child_name="castor_rightleft" mass="${castor_mass}" length="0.045" radius="0.04" ox="0.0" oy="-0.0225" oz="-0.075" roll="${pi/2}" yaw="0.0" pitch="0.0" color="Grey" mu1="${mu1}" mu2="${mu2}" kp="${kp}" kd="${kd}"  />
+  <xacro:default_zylinder_in_Y_with_collision parent="castor_plate_right" child_name="castor_leftright" mass="${castor_mass}" length="0.045" radius="0.04" ox="0.0" oy="0.0225" oz="-0.075" roll="${pi/2}" yaw="0.0" pitch="0.0" color="Grey" mu1="${mu1}" mu2="${mu2}" kp="${kp}" kd="${kd}"  />
+  <xacro:default_zylinder_in_Y_with_collision parent="castor_plate_right" child_name="castor_rightright" mass="${castor_mass}" length="0.045" radius="0.04" ox="0.0" oy="-0.0225" oz="-0.075" roll="${pi/2}" yaw="0.0" pitch="0.0" color="Grey" mu1="${mu1}" mu2="${mu2}" kp="${kp}" kd="${kd}"  />
   <!-- //////////////////////////////////////////////////////////////////////////// -->
   <!-- ////////////////////////// Actuators and Sensors ////////////////////////// -->
@@ -108,5 +108,5 @@
       <updateRate>50.0</updateRate>
       <bodyName>base_link</bodyName>
-      <topicName>imu/data</topicName>
+      <topicName>imu/data_raw</topicName>
       <accelDrift>0.005 0.005 0.005</accelDrift>
       <accelGaussianNoise>0.005 0.005 0.005</accelGaussianNoise>

File: beaverbot_description/urdf/beaverbot.xacro (robot description, xacro)
@@ -163,5 +163,5 @@
     </joint>
   </xacro:macro>
-  <xacro:macro name="default_zylinder_in_Y_with_collision" params="parent child_name mass length radius ox oy oz roll pitch yaw color">
+  <xacro:macro name="default_zylinder_in_Y_with_collision" params="parent child_name mass length radius ox oy oz roll pitch yaw color mu1 mu2 kp kd">
     <link name="${child_name}" >
       <visual>
@@ -181,4 +181,8 @@
     </link>
     <gazebo reference="${child_name}" >
+      <mu1 value="${mu1}"/>
+      <mu2 value="${mu2}"/>
+      <kp value="${kp}" />
+      <kd value="${kd}" />
       <material>Gazebo/${color}</material>
     </gazebo>

Commit message: :+1: modify imu and implement gps

File: beaverbot_description/urdf/beaverbot.urdf.xacro (robot description, xacro)
@@ -95,5 +95,5 @@
   <xacro:wheel_actuator parent="wheel_support_right" child_name="wheel_right" mass="${wheel_mass}" length="0.06" radius="${wheel_radius}" ox="0.0" oy="-0.095" oz="0.0" roll="${pi/2}" yaw="0.0" pitch="0.0" color="Grey" axis_x="0" axis_y="1" axis_z="0" mu1="${mu1}" mu2="${mu2}" kp="${kp}" kd="${kd}" />
   <xacro:lidar_sensor parent="lidar_base" lidar_name="laser" length="${lidar_length}" radius="${lidar_radius}" mass="${lidar_mass}" ox="0.0" oy="0.0" oz="0.0325" update_rate="${lidar_update_rate}" min_angle="${lidar_min_angle}" max_angle="${lidar_max_angle}" min_range="${lidar_min_range}" max_range="${lidar_max_range}" range_resolution="${lidar_range_resolution}" stdv="${lidar_stdv}" />
-  <xacro:imu_sensor parent="back_base_support_frame" imu_name="imu_sensor" mass="${imu_mass}" sizex="0.03" sizey="0.03" sizez="0.005" ox="0.0" oy="0.0" oz="0.01" update_rate="${imu_update_rate}" update_rateHz="${imu_update_rateHz}" noise="${imu_noise}" />
+  <xacro:imu_sensor parent="back_base_support_frame" imu_name="imu" imu_topic="imu/data_raw" mass="${imu_mass}" sizex="0.03" sizey="0.03" sizez="0.005" ox="0.0" oy="0.0" oz="0.01" update_rate="${imu_update_rate}" update_rateHz="${imu_update_rateHz}" noise="${imu_noise}" />
   <!-- /////////////////////////////////////////////////////////////////////////// -->
  <gazebo>
@@ -103,32 +103,3 @@
     </plugin>
   </gazebo>
-  <gazebo>
-    <plugin name="imu_controller" filename="libhector_gazebo_ros_imu.so">
-      <robotNamespace>$(arg robot_namespace)</robotNamespace>
-      <updateRate>50.0</updateRate>
-      <bodyName>base_link</bodyName>
-      <topicName>imu/data_raw</topicName>
-      <accelDrift>0.005 0.005 0.005</accelDrift>
-      <accelGaussianNoise>0.005 0.005 0.005</accelGaussianNoise>
-      <rateDrift>0.005 0.005 0.005 </rateDrift>
-      <rateGaussianNoise>0.005 0.005 0.005 </rateGaussianNoise>
-      <headingDrift>0.005</headingDrift>
-      <headingGaussianNoise>0.005</headingGaussianNoise>
-    </plugin>
-  </gazebo>
-  <gazebo>
-    <plugin name="gps_controller" filename="libhector_gazebo_ros_gps.so">
-      <robotNamespace>$(arg robot_namespace)</robotNamespace>
-      <updateRate>40</updateRate>
-      <bodyName>base_link</bodyName>
-      <frameId>map</frameId>
-      <topicName>navsat/fix</topicName>
-      <velocityTopicName>navsat/vel</velocityTopicName>
-      <referenceLatitude>34.835190564394</referenceLatitude>
-      <referenceLongitude>137.45711512765206</referenceLongitude>
-      <referenceHeading>0</referenceHeading>
-      <referenceAltitude>0</referenceAltitude>
-      <drift>0.0001 0.0001 0.0001</drift>
-    </plugin>
-  </gazebo>
 </robot>

File: beaverbot_description/urdf/sensors_and_actuators.xacro (robot description, xacro)
@@ -219,43 +219,82 @@
     </gazebo>
   </xacro:macro>
-<!-- /////////////////////////////////////////////////////////////////// -->
-<!-- ////////////////////////////// IMU ////////////////////////////// -->
-  <xacro:macro name="imu_sensor" params="parent imu_name mass sizex sizey sizez ox oy oz update_rate update_rateHz noise" >
+	<!-- /////////////////////////////////////////////////////////////////// -->
+	<!-- ////////////////////////////// IMU ////////////////////////////// -->
+  <xacro:macro name="imu_sensor" params="parent imu_name imu_topic mass sizex sizey sizez ox oy oz update_rate update_rateHz noise" >
     <link name="${imu_name}">
+			<visual>
+				<geometry>
+					<box size="${sizex} ${sizey} ${sizez}"/>
+				</geometry>
+				<material name="White"/>
+			</visual>
+			<xacro:inertial_box mass="${mass}" x="${sizex}" y="${sizey}" z="${sizez}" />
+    </link>
+		<joint name="${parent}_to_${imu_name}" type="fixed">
+			<parent link="${parent}"/>
+			<child link="${imu_name}"/>
+			<origin xyz="${ox} ${oy} ${oz}"/>
+		</joint>
+    <gazebo reference="${imu_name}">
+      <material>Gazebo/White</material>
+			<gravity>true</gravity>
+			<sensor name="${imu_name}_sensor" type="imu">
+				<always_on>true</always_on>
+				<update_rate>${update_rate}</update_rate>
+				<visualize>true</visualize>
+				<topic>${imu_topic}</topic>
+				<plugin filename="libgazebo_ros_imu_sensor.so" name="imu_plugin">
+					<topicName>${imu_topic}</topicName>
+					<bodyName>${imu_name}</bodyName>
+					<updateRateHZ>${update_rateHz}</updateRateHZ>
+					<gaussianNoise>${noise}</gaussianNoise>
+					<xyzOffset>0 0 0</xyzOffset>
+					<rpyOffset>0 0 0</rpyOffset>
+					<frameName>${imu_name}</frameName>
+				</plugin>
+				<pose>0 0 0 0 0 0</pose>
+			</sensor>
+    </gazebo>
+  </xacro:macro>
+	<!-- ///////////////////////////////////////////////////////////////// -->
+	<!-- ////////////////////////////GPS SENSORS//////////////////////////// -->
+  <xacro:macro name="gps_sensor" params="parent gps_name mass sizex sizey sizez ox oy oz update_rate update_rateHz noise">
+	<link name="${gps_name}">
 	  <visual>
 	    <geometry>
 	      <box size="${sizex} ${sizey} ${sizez}"/>
 		</geometry>
-	    <material name="White"/>
+		<material name="White"/>
 	  </visual>
 	  <xacro:inertial_box mass="${mass}" x="${sizex}" y="${sizey}" z="${sizez}" />
-    </link>
-	<joint name="${parent}_to_${imu_name}" type="fixed">
+	</link>
+	<joint name="${parent}_to_${gps_name}" type="fixed">
 	  <parent link="${parent}"/>
-	  <child link="${imu_name}"/>
+	  <child link="${gps_name}"/>
 	  <origin xyz="${ox} ${oy} ${oz}"/>
 	</joint>
-        <!-- maybe switch to the Hector version of the IMU -->
-    <gazebo reference="${imu_name}">
-      <material>Gazebo/White</material>
+	<gazebo reference="${gps_name}">
+		<material>Gazebo/White</material>
 	  <gravity>true</gravity>
-	  <sensor name="${imu_name}_sensor" type="imu">
-	    <always_on>true</always_on>
+	  <sensor name="${gps_name}_sensor" type="gps">
+			<always_on>true</always_on>
 	    <update_rate>${update_rate}</update_rate>
 	    <visualize>true</visualize>
-	    <topic>__default_topic__</topic>
-  		<plugin filename="libgazebo_ros_imu_sensor.so" name="imu_plugin">
-		  <topicName>imu</topicName>
-                  <bodyName>${imu_name}</bodyName>
-		  <updateRateHZ>${update_rateHz}</updateRateHZ>
-                  <gaussianNoise>${noise}</gaussianNoise>
-		  <xyzOffset>0 0 0</xyzOffset>
-		  <rpyOffset>0 0 0</rpyOffset>
-                  <frameName>${imu_name}</frameName>
-	    </plugin>
-	    <pose>0 0 0 0 0 0</pose>
-	  </sensor>
-    </gazebo>
-  </xacro:macro>
-<!-- ///////////////////////////////////////////////////////////////// -->
+	    <topic>${imu_topic}</topic>
+		<plugin name="gps_controller" filename="libhector_gazebo_ros_gps.so">
+			<robotNamespace>$(arg robot_namespace)</robotNamespace>
+		  <updateRate>40</updateRate>
+			<bodyName>base_link</bodyName>
+			<frameId>map</frameId>
+			<topicName>navsat/fix</topicName>
+			<velocityTopicName>navsat/vel</velocityTopicName>
+			<referenceLatitude>34.835190564394</referenceLatitude>
+			<referenceLongitude>137.45711512765206</referenceLongitude>
+			<referenceHeading>0</referenceHeading>
+			<referenceAltitude>0</referenceAltitude>
+			<drift>0.0001 0.0001 0.0001</drift>
+		</plugin>
+			</sensor>
+	</gazebo>
+	</xacro:macro>
 </robot>

Commit message: :+1: update gps and imu

File: beaverbot_description/urdf/beaverbot.urdf.xacro (robot description, xacro)
@@ -95,5 +95,6 @@
   <xacro:wheel_actuator parent="wheel_support_right" child_name="wheel_right" mass="${wheel_mass}" length="0.06" radius="${wheel_radius}" ox="0.0" oy="-0.095" oz="0.0" roll="${pi/2}" yaw="0.0" pitch="0.0" color="Grey" axis_x="0" axis_y="1" axis_z="0" mu1="${mu1}" mu2="${mu2}" kp="${kp}" kd="${kd}" />
   <xacro:lidar_sensor parent="lidar_base" lidar_name="laser" length="${lidar_length}" radius="${lidar_radius}" mass="${lidar_mass}" ox="0.0" oy="0.0" oz="0.0325" update_rate="${lidar_update_rate}" min_angle="${lidar_min_angle}" max_angle="${lidar_max_angle}" min_range="${lidar_min_range}" max_range="${lidar_max_range}" range_resolution="${lidar_range_resolution}" stdv="${lidar_stdv}" />
-  <xacro:imu_sensor parent="back_base_support_frame" imu_name="imu" imu_topic="imu/data_raw" mass="${imu_mass}" sizex="0.03" sizey="0.03" sizez="0.005" ox="0.0" oy="0.0" oz="0.01" update_rate="${imu_update_rate}" update_rateHz="${imu_update_rateHz}" noise="${imu_noise}" />
+  <xacro:imu_sensor parent="back_base_support_frame" imu_name="imu" imu_topic="imu/data_raw" mass="${imu_mass}" sizex="0.03" sizey="0.03" sizez="0.005" ox="0.0" oy="0.0" oz="0.01" update_rate="${imu_update_rate}" noise="${imu_noise}" />
+  <xacro:gps_sensor parent="back_base_support_frame" gps_name="gps" gps_topic="gps/fix" mass="${gps_mass}" sizex="0.03" sizey="0.03" sizez="0.005" ox="0.0" oy="0.0" oz="0.0015" update_rate="${gps_update_rate}" initial_latitude="${gps_latitude}" initial_longitude="${gps_longitude}" noise="${gps_noise}" />
   <!-- /////////////////////////////////////////////////////////////////////////// -->
  <gazebo>

File: beaverbot_description/urdf/properties.xacro (robot description, xacro)
@@ -43,8 +43,12 @@
   <xacro:property name="lidar_min_angle" value="0.0" />
   <xacro:property name="lidar_max_angle" value="6.283185" />
-  <xacro:property name="imu_update_rate" value="25.0" />			<!-- update rate in ms -->
-  <xacro:property name="imu_update_rateHz" value="40.0" />
+  <xacro:property name="imu_update_rate" value="40.0" />
   <xacro:property name="imu_mass" value="0.05" />
   <xacro:property name="imu_noise" value="0.001" />
+  <xacro:property name="gps_update_rate" value="10.0" />
+  <xacro:property name="gps_mass" value="0.05" />
+  <xacro:property name="gps_noise" value="0.001" />
+  <xacro:property name="gps_latitude" value="34.835190564394" />
+  <xacro:property name="gps_longitude" value="137.45711512765206" />
   <xacro:property name="mu1" value="0.6" />
   <xacro:property name="mu2" value="0.6" />

File: beaverbot_description/urdf/sensors_and_actuators.xacro (robot description, xacro)
@@ -221,43 +221,43 @@
 	<!-- /////////////////////////////////////////////////////////////////// -->
 	<!-- ////////////////////////////// IMU ////////////////////////////// -->
-  <xacro:macro name="imu_sensor" params="parent imu_name imu_topic mass sizex sizey sizez ox oy oz update_rate update_rateHz noise" >
+  <xacro:macro name="imu_sensor" params="parent imu_name imu_topic mass sizex sizey sizez ox oy oz update_rate noise" >
     <link name="${imu_name}">
-			<visual>
-				<geometry>
-					<box size="${sizex} ${sizey} ${sizez}"/>
-				</geometry>
-				<material name="White"/>
-			</visual>
-			<xacro:inertial_box mass="${mass}" x="${sizex}" y="${sizey}" z="${sizez}" />
+	<visual>
+		<geometry>
+			<box size="${sizex} ${sizey} ${sizez}"/>
+		</geometry>
+		<material name="White"/>
+	</visual>
+	<xacro:inertial_box mass="${mass}" x="${sizex}" y="${sizey}" z="${sizez}" />
     </link>
-		<joint name="${parent}_to_${imu_name}" type="fixed">
-			<parent link="${parent}"/>
-			<child link="${imu_name}"/>
-			<origin xyz="${ox} ${oy} ${oz}"/>
-		</joint>
-    <gazebo reference="${imu_name}">
-      <material>Gazebo/White</material>
-			<gravity>true</gravity>
-			<sensor name="${imu_name}_sensor" type="imu">
-				<always_on>true</always_on>
-				<update_rate>${update_rate}</update_rate>
-				<visualize>true</visualize>
-				<topic>${imu_topic}</topic>
-				<plugin filename="libgazebo_ros_imu_sensor.so" name="imu_plugin">
-					<topicName>${imu_topic}</topicName>
-					<bodyName>${imu_name}</bodyName>
-					<updateRateHZ>${update_rateHz}</updateRateHZ>
-					<gaussianNoise>${noise}</gaussianNoise>
-					<xyzOffset>0 0 0</xyzOffset>
-					<rpyOffset>0 0 0</rpyOffset>
-					<frameName>${imu_name}</frameName>
-				</plugin>
-				<pose>0 0 0 0 0 0</pose>
-			</sensor>
-    </gazebo>
+	<joint name="${parent}_to_${imu_name}" type="fixed">
+		<parent link="${parent}"/>
+		<child link="${imu_name}"/>
+		<origin xyz="${ox} ${oy} ${oz}"/>
+	</joint>
+	<gazebo reference="${imu_name}">
+		<material>Gazebo/White</material>
+		<gravity>true</gravity>
+		<sensor name="${imu_name}_sensor" type="imu">
+			<always_on>true</always_on>
+			<update_rate>${update_rate}</update_rate>
+			<visualize>true</visualize>
+			<topic>${imu_topic}</topic>
+			<plugin filename="libgazebo_ros_imu_sensor.so" name="imu_plugin">
+				<topicName>${imu_topic}</topicName>
+				<bodyName>${imu_name}</bodyName>
+				<updateRate>${update_rate}</updateRate>
+				<gaussianNoise>${noise}</gaussianNoise>
+				<xyzOffset>0 0 0</xyzOffset>
+				<rpyOffset>0 0 0</rpyOffset>
+				<frameName>${imu_name}</frameName>
+			</plugin>
+			<pose>0 0 0 0 0 0</pose>
+		</sensor>
+	</gazebo>
   </xacro:macro>
 	<!-- ///////////////////////////////////////////////////////////////// -->
 	<!-- ////////////////////////////GPS SENSORS//////////////////////////// -->
-  <xacro:macro name="gps_sensor" params="parent gps_name mass sizex sizey sizez ox oy oz update_rate update_rateHz noise">
+  <xacro:macro name="gps_sensor" params="parent gps_name gps_topic mass sizex sizey sizez ox oy oz update_rate initial_latitude initial_longitude noise">
 	<link name="${gps_name}">
 	  <visual>
@@ -274,26 +274,17 @@
 	  <origin xyz="${ox} ${oy} ${oz}"/>
 	</joint>
-	<gazebo reference="${gps_name}">
-		<material>Gazebo/White</material>
-	  <gravity>true</gravity>
-	  <sensor name="${gps_name}_sensor" type="gps">
-			<always_on>true</always_on>
-	    <update_rate>${update_rate}</update_rate>
-	    <visualize>true</visualize>
-	    <topic>${imu_topic}</topic>
-		<plugin name="gps_controller" filename="libhector_gazebo_ros_gps.so">
-			<robotNamespace>$(arg robot_namespace)</robotNamespace>
-		  <updateRate>40</updateRate>
-			<bodyName>base_link</bodyName>
-			<frameId>map</frameId>
-			<topicName>navsat/fix</topicName>
+	<gazebo>
+		<plugin filename="libhector_gazebo_ros_gps.so" name="gps_plugin">
+			<updateRate>${update_rate}</updateRate>
+			<bodyName>${gps_name}</bodyName>
+			<frameId>${gps_name}</frameId>
+			<topicName>${gps_topic}</topicName>
 			<velocityTopicName>navsat/vel</velocityTopicName>
-			<referenceLatitude>34.835190564394</referenceLatitude>
-			<referenceLongitude>137.45711512765206</referenceLongitude>
+			<referenceLatitude>${initial_latitude}</referenceLatitude>
+			<referenceLongitude>${initial_longitude}</referenceLongitude>
 			<referenceHeading>0</referenceHeading>
 			<referenceAltitude>0</referenceAltitude>
-			<drift>0.0001 0.0001 0.0001</drift>
+			<gaussianNoise>${noise}</gaussianNoise>
 		</plugin>
-			</sensor>
 	</gazebo>
 	</xacro:macro>
