Commit message: :+1: implement trailer-tractor

File: beaverbot_description/urdf/beaverbot.urdf.xacro (robot description, xacro)
@@ -97,4 +97,7 @@
   <xacro:imu_sensor parent="back_base_support_frame" imu_name="imu" imu_topic="imu/data_raw" mass="${imu_mass}" sizex="0.03" sizey="0.03" sizez="0.005" ox="0.0" oy="0.0" oz="0.01" update_rate="${imu_update_rate}" noise="${imu_noise}" />
   <xacro:gps_sensor parent="back_base_support_frame" gps_name="gps" gps_topic="gps/fix" mass="${gps_mass}" sizex="0.03" sizey="0.03" sizez="0.005" ox="0.0" oy="0.0" oz="0.0015" update_rate="${gps_update_rate}" initial_latitude="${gps_latitude}" initial_longitude="${gps_longitude}" noise="${gps_noise}" />
+  <xacro:if value="${use_trailer}">
+    <xacro:trailer parent="base" trailer_name="trailer" mu1="0.1" mu2="0.1" kp="${kp}" kd="${kd}" />
+  </xacro:if>
   <!-- /////////////////////////////////////////////////////////////////////////// -->
  <gazebo>

File: beaverbot_description/urdf/properties.xacro (robot description, xacro)
@@ -51,8 +51,9 @@
   <xacro:property name="gps_latitude" value="34.835190564394" />
   <xacro:property name="gps_longitude" value="137.45711512765206" />
-  <xacro:property name="mu1" value="0.6" />
-  <xacro:property name="mu2" value="0.6" />
+  <xacro:property name="mu1" value="0.1" />
+  <xacro:property name="mu2" value="0.1" />
   <xacro:property name="kp" value="10000000.0" />
-  <xacro:property name="kd" value="40.0" />
+  <xacro:property name="kd" value="1.0" />
+  <xacro:property name="use_trailer" value="true" />
   <!-- ///////////////////////////////////////////////////////////// -->
 </robot>

File: beaverbot_description/urdf/sensors_and_actuators.xacro (robot description, xacro)
@@ -161,4 +161,132 @@
   </xacro:macro>
 <!-- /////////////////////////////////////////////////////////////////// -->
+<!-- ////////////////////////////// Trailer ////////////////////////////// -->
+<xacro:macro name="trailer" params="parent trailer_name mu1 mu2 kp kd">
+	<link name="${trailer_name}_base_link">
+		<visual>
+			<geometry>
+				<box size="0.01 0.01 0.01"/>
+			</geometry>
+		</visual>
+		<collision>
+			<geometry>
+				<box size="0.01 0.01 0.01"/>
+			</geometry>
+		</collision>
+		<xacro:inertial_box mass="0.001" x="0.01" y="0.01" z="0.01" />
+	</link>
+	<gazebo reference="${trailer_name}_base_link" >
+	  <material>Gazebo/White</material>
+	</gazebo>
+	<link name="${trailer_name}_connector">
+		<visual>
+			<origin xyz="-0.25 0 0" rpy="0 0 0" />
+			<geometry>
+				<box size="0.5 0.05 0.01"/>
+			</geometry>
+		</visual>
+		<collision>
+			<origin xyz="-0.25 0 0" rpy="0 0 0" />
+			<geometry>
+				<box size="0.5 0.05 0.01"/>
+			</geometry>
+		</collision>
+		<xacro:inertial_box mass="0.001" x="0.01" y="0.01" z="0.01" />
+	</link>
+	<link name="tractor_connector">
+		<visual>
+			<origin xyz="0.15 0 0" rpy="0 0 0" />
+			<geometry>
+				<box size="0.3 0.05 0.01"/>
+			</geometry>
+		</visual>
+		<collision>
+			<origin xyz="0.15 0 0" rpy="0 0 0" />
+			<geometry>
+				<box size="0.3 0.05 0.01"/>
+			</geometry>
+		</collision>
+		<xacro:inertial_box mass="0.001" x="0.01" y="0.01" z="0.01" />
+	</link>
+	<gazebo reference="tractor_connector" >
+		<material>Gazebo/White</material>
+	</gazebo>
+	<joint name="tractor_to_${parent}" type="fixed">
+		<parent link="${parent}" />
+		<child link="tractor_connector" />
+		<origin xyz="-0.45 0 0" rpy="0 0 0" />
+	</joint>
+	<joint name="tractor_connector_to_trailer_connector" type="revolute">
+		<parent link="tractor_connector" />
+		<child link="${trailer_name}_connector" />
+		<origin xyz="0.0 0.0 0.0" rpy="0.0 0.0 0.0" />
+		<axis xyz="0 0 1" />
+		<limit lower="-${pi/4.0}" upper="${pi/4.0}" effort="1.0" velocity="0.01"/>
+		<dynamics damping="0.01" friction="0.01"/>
+	</joint>
+	<joint name="${trailer_name}_connector_to_${trailer_name}_base_link" type="fixed">
+		<parent link="${trailer_name}_connector" />
+		<child link="${trailer_name}_base_link" />
+		<origin xyz="-0.5 0 0" rpy="0 0 0" />
+	</joint>
+	<xacro:default_zylinder_in_Y parent="${trailer_name}_base_link" child_name="${trailer_name}_wheel_support_left" mass="0.01" length="0.13" radius="0.05" ox="0.0" oy="0.155" oz="-0.061" roll="1.57" yaw="0.0" pitch="0.0" color="White" />
+	<xacro:default_zylinder_in_Y parent="${trailer_name}_base_link" child_name="${trailer_name}_wheel_support_right" mass="0.01" length="0.13" radius="0.05" ox="0.0" oy="-0.155" oz="-0.061" roll="1.57" yaw="0.0" pitch="0.0" color="White" />
+	<link name="${trailer_name}_left_wheel">
+		<visual>
+			<geometry>
+				<cylinder length="0.05" radius="0.164" />
+			</geometry>
+			<origin xyz="0 0 0" rpy="1.57 0 0" />
+		</visual>
+		<collision>
+			<geometry>
+				<cylinder length="0.05" radius="0.164" />
+			</geometry>
+			<origin xyz="0 0 0" rpy="1.57 0 0" />
+		</collision>
+		<xacro:inertial_zylinder_y mass="0.01" radius="0.164" height="0.01" />
+	</link>
+	<joint name="${trailer_name}_wheel_shaft_to_left_wheel" type="continuous">
+		<parent link="${trailer_name}_wheel_support_left" />
+		<child link="${trailer_name}_left_wheel" />
+		<origin xyz="0 0.095 0" rpy="0 0 0" />
+		<axis xyz="0 1 0" />
+	</joint>
+	<link name="${trailer_name}_right_wheel">
+		<visual>
+			<geometry>
+				<cylinder length="0.05" radius="0.164" />
+			</geometry>
+			<origin xyz="0 0 0" rpy="1.57 0 0" />
+		</visual>
+		<collision>
+			<geometry>
+				<cylinder length="0.05" radius="0.164" />
+			</geometry>
+			<origin xyz="0 0 0" rpy="1.57 0 0" />
+		</collision>
+		<xacro:inertial_zylinder_y mass="0.01" radius="0.164" height="0.05" />
+	</link>
+	<joint name="${trailer_name}_wheel_shaft_to_right_wheel" type="continuous">
+		<parent link="${trailer_name}_wheel_support_right" />
+		<child link="${trailer_name}_right_wheel" />
+		<origin xyz="0 -0.095 0" rpy="0 0 0" />
+		<axis xyz="0 1 0" />
+	</joint>
+	<gazebo reference="${trailer_name}_left_wheel" >
+      <mu1 value="${mu1}"/>
+      <mu2 value="${mu2}"/>
+      <kp value="${kp}" />
+      <kd value="${kd}" />
+      <material>Gazebo/White</material>
+    </gazebo>
+    <gazebo reference="${trailer_name}_right_wheel" >
+      <mu1 value="${mu1}"/>
+      <mu2 value="${mu2}"/>
+      <kp value="${kp}" />
+      <kd value="${kd}" />
+      <material>Gazebo/White</material>
+    </gazebo>
+  </xacro:macro>
 <!-- ////////////////////////////// Lidar ////////////////////////////// -->
   <xacro:macro name="lidar_sensor" params="parent lidar_name length radius mass ox oy oz update_rate min_angle max_angle min_range max_range range_resolution stdv" >

Commit message: :+1: update cleaner

File: beaverbot_description/urdf/beaverbot.urdf.xacro (robot description, xacro)
@@ -23,5 +23,5 @@
       </geometry>
     </collision>
-    <xacro:inertial_box mass="0.01" x="0.01" y="0.01" z="0.01" />
+    <xacro:inertial_box mass="0.01" x="0.01" y="0.01" z="0.01" ox="0.0" oy="0.0" oz="0.0"/>
   </link>
   <gazebo reference="base_link">
@@ -35,5 +35,5 @@
       <material name="Black"/>
     </visual>
-    <xacro:inertial_box mass="${base_mass}" x="0.52" y="0.21" z="0.21" />
+    <xacro:inertial_box mass="${base_mass}" x="0.52" y="0.21" z="0.21" ox="0.0" oy="0.0" oz="0.0"/>
   </link>
   <gazebo reference="base">

File: beaverbot_description/urdf/beaverbot.xacro (robot description, xacro)
@@ -21,6 +21,7 @@
     </inertial>
   </xacro:macro>
-  <xacro:macro name="inertial_box" params="mass x y z">
-    <inertial>
+  <xacro:macro name="inertial_box" params="mass x y z ox oy oz">
+    <inertial>
+      <origin xyz="${ox} ${oy} ${oz}" />
       <mass value="${mass}" />
       <inertia ixx="${(mass/12)*(y*y+z*z)}" ixy="0.0" ixz="0.0" iyy="${(mass/12)*(x*x+z*z)}" iyz="0.0" izz="${(mass/12)*(y*y+x*x)}" />
@@ -38,5 +39,5 @@
         <material name="${color}" />
       </visual>
-      <xacro:inertial_box mass="${mass}" x="${sizex}" y="${sizey}" z="${sizez}" />
+      <xacro:inertial_box mass="${mass}" x="${sizex}" y="${sizey}" z="${sizez}" ox="0.0" oy="0.0" oz="0.0" />
     </link>
     <gazebo reference="${child_name}" >
@@ -126,5 +127,5 @@
         <origin rpy="${roll} ${pitch} ${yaw}" />
       </collision>
-      <xacro:inertial_box mass="${mass}" x="${sizex}" y="${sizey}" z="${sizez}" />
+      <xacro:inertial_box mass="${mass}" x="${sizex}" y="${sizey}" z="${sizez}" ox="0.0" oy="0.0" oz="0.0"/>
     </link>
     <gazebo reference="${child_name}" >

File: beaverbot_description/urdf/properties.xacro (robot description, xacro)
@@ -51,6 +51,6 @@
   <xacro:property name="gps_latitude" value="34.835190564394" />
   <xacro:property name="gps_longitude" value="137.45711512765206" />
-  <xacro:property name="mu1" value="0.1" />
-  <xacro:property name="mu2" value="0.1" />
+  <xacro:property name="mu1" value="0.5" />
+  <xacro:property name="mu2" value="0.5" />
   <xacro:property name="kp" value="10000000.0" />
   <xacro:property name="kd" value="1.0" />

File: beaverbot_description/urdf/sensors_and_actuators.xacro (robot description, xacro)
@@ -10,5 +10,5 @@
 		<material name="White" />
 	  </visual>
-	  <xacro:inertial_box mass="${mass}" x="${sizex}" y="${sizey}" z="${sizez}" />
+	  <xacro:inertial_box mass="${mass}" x="${sizex}" y="${sizey}" z="${sizez}" ox="0.0" oy="0.0" oz="0.0"/>
 	</link>
         <joint name="${parent}_to_${prefix}_${sufix}" type="fixed">
@@ -71,5 +71,5 @@
 		<material name="White" />
 	  </visual>
-	  <xacro:inertial_box mass="${mass}" x="${dist_size}" y="${dist_size}" z="${dist_size}" />
+	  <xacro:inertial_box mass="${mass}" x="${dist_size}" y="${dist_size}" z="${dist_size}" ox="0.0" oy="0.0" oz="0.0"/>
 	</link>
 	<gazebo reference="${prefix}_distance_sensor_link_${sufix}">
@@ -166,16 +166,18 @@
 		<visual>
 			<geometry>
-				<box size="0.01 0.01 0.01"/>
-			</geometry>
+				<mesh filename="package://beaverbot_description/meshes/cleaner.stl" scale="0.001 0.001 0.001"/>
+			</geometry>
+			<origin rpy="1.57 0 -1.57" xyz="-0.15 0.4 -0.05" />
 		</visual>
 		<collision>
 			<geometry>
-				<box size="0.01 0.01 0.01"/>
-			</geometry>
+				<mesh filename="package://beaverbot_description/meshes/cleaner.stl" scale="0.001 0.001 0.001"/>
+			</geometry>
+			<origin rpy="1.57 0 -1.57" xyz="-0.15 0.4 -0.05" />
 		</collision>
-		<xacro:inertial_box mass="0.001" x="0.01" y="0.01" z="0.01" />
+		<xacro:inertial_box mass="0.001" x="0.01" y="0.01" z="0.01" ox="-0.15" oy="0.4" oz="-0.05"/>
 	</link>
 	<gazebo reference="${trailer_name}_base_link" >
-	  <material>Gazebo/White</material>
+	  <material>Gazebo/Gray</material>
 	</gazebo>
 	<link name="${trailer_name}_connector">
@@ -192,6 +194,9 @@
 			</geometry>
 		</collision>
-		<xacro:inertial_box mass="0.001" x="0.01" y="0.01" z="0.01" />
-	</link>
+		<xacro:inertial_box mass="0.001" x="0.01" y="0.01" z="0.01" ox="0.0" oy="0.0" oz="0.0"/>
+	</link>
+	<gazebo reference="${trailer_name}_connector" >
+		<material>Gazebo/DarkGray</material>
+	</gazebo>
 	<link name="tractor_connector">
 		<visual>
@@ -207,13 +212,13 @@
 			</geometry>
 		</collision>
-		<xacro:inertial_box mass="0.001" x="0.01" y="0.01" z="0.01" />
+		<xacro:inertial_box mass="0.01" x="0.01" y="0.01" z="0.01" ox="0.0" oy="0.0" oz="0.0"/>
 	</link>
 	<gazebo reference="tractor_connector" >
-		<material>Gazebo/White</material>
+		<material>Gazebo/DarkGray</material>
 	</gazebo>
 	<joint name="tractor_to_${parent}" type="fixed">
 		<parent link="${parent}" />
 		<child link="tractor_connector" />
-		<origin xyz="-0.45 0 0" rpy="0 0 0" />
+		<origin xyz="-0.45 0 -0.1" rpy="0 0 0" />
 	</joint>
 	<joint name="tractor_connector_to_trailer_connector" type="revolute">
@@ -223,17 +228,17 @@
 		<axis xyz="0 0 1" />
 		<limit lower="-${pi/4.0}" upper="${pi/4.0}" effort="1.0" velocity="0.01"/>
-		<dynamics damping="0.01" friction="0.01"/>
+		<dynamics damping="0.001" friction="0.001"/>
 	</joint>
 	<joint name="${trailer_name}_connector_to_${trailer_name}_base_link" type="fixed">
 		<parent link="${trailer_name}_connector" />
 		<child link="${trailer_name}_base_link" />
-		<origin xyz="-0.5 0 0" rpy="0 0 0" />
-	</joint>
-	<xacro:default_zylinder_in_Y parent="${trailer_name}_base_link" child_name="${trailer_name}_wheel_support_left" mass="0.01" length="0.13" radius="0.05" ox="0.0" oy="0.155" oz="-0.061" roll="1.57" yaw="0.0" pitch="0.0" color="White" />
-	<xacro:default_zylinder_in_Y parent="${trailer_name}_base_link" child_name="${trailer_name}_wheel_support_right" mass="0.01" length="0.13" radius="0.05" ox="0.0" oy="-0.155" oz="-0.061" roll="1.57" yaw="0.0" pitch="0.0" color="White" />
+		<origin xyz="-1 0 0" rpy="0 0 0" />
+	</joint>
+	<xacro:default_zylinder_in_Y parent="${trailer_name}_base_link" child_name="${trailer_name}_wheel_support_left" mass="0.001" length="0.1" radius="0.05" ox="0.0" oy="0.32" oz="-0.0" roll="1.57" yaw="0.0" pitch="0.0" color="White" />
+	<xacro:default_zylinder_in_Y parent="${trailer_name}_base_link" child_name="${trailer_name}_wheel_support_right" mass="0.001" length="0.1" radius="0.05" ox="0.0" oy="-0.32" oz="-0.0" roll="1.57" yaw="0.0" pitch="0.0" color="White" />
 	<link name="${trailer_name}_left_wheel">
 		<visual>
 			<geometry>
-				<cylinder length="0.05" radius="0.164" />
+				<cylinder length="0.05" radius="0.114" />
 			</geometry>
 			<origin xyz="0 0 0" rpy="1.57 0 0" />
@@ -241,9 +246,9 @@
 		<collision>
 			<geometry>
-				<cylinder length="0.05" radius="0.164" />
+				<cylinder length="0.05" radius="0.114" />
 			</geometry>
 			<origin xyz="0 0 0" rpy="1.57 0 0" />
 		</collision>
-		<xacro:inertial_zylinder_y mass="0.01" radius="0.164" height="0.01" />
+		<xacro:inertial_zylinder_y mass="0.01" radius="0.114" height="0.01" />
 	</link>
 	<joint name="${trailer_name}_wheel_shaft_to_left_wheel" type="continuous">
@@ -256,5 +261,5 @@
 		<visual>
 			<geometry>
-				<cylinder length="0.05" radius="0.164" />
+				<cylinder length="0.05" radius="0.114" />
 			</geometry>
 			<origin xyz="0 0 0" rpy="1.57 0 0" />
@@ -262,9 +267,9 @@
 		<collision>
 			<geometry>
-				<cylinder length="0.05" radius="0.164" />
+				<cylinder length="0.05" radius="0.114" />
 			</geometry>
 			<origin xyz="0 0 0" rpy="1.57 0 0" />
 		</collision>
-		<xacro:inertial_zylinder_y mass="0.01" radius="0.164" height="0.05" />
+		<xacro:inertial_zylinder_y mass="0.01" radius="0.114" height="0.05" />
 	</link>
 	<joint name="${trailer_name}_wheel_shaft_to_right_wheel" type="continuous">
@@ -279,5 +284,5 @@
       <kp value="${kp}" />
       <kd value="${kd}" />
-      <material>Gazebo/White</material>
+      <material>Gazebo/DarkGray</material>
     </gazebo>
     <gazebo reference="${trailer_name}_right_wheel" >
@@ -286,5 +291,5 @@
       <kp value="${kp}" />
       <kd value="${kd}" />
-      <material>Gazebo/White</material>
+      <material>Gazebo/DarkGray</material>
     </gazebo>
   </xacro:macro>
@@ -356,5 +361,5 @@
 		<material name="White"/>
 	</visual>
-	<xacro:inertial_box mass="${mass}" x="${sizex}" y="${sizey}" z="${sizez}" />
+	<xacro:inertial_box mass="${mass}" x="${sizex}" y="${sizey}" z="${sizez}" ox="0.0" oy="0.0" oz="0.0"/>
     </link>
 	<joint name="${parent}_to_${imu_name}" type="fixed">
@@ -394,5 +399,5 @@
 		<material name="White"/>
 	  </visual>
-	  <xacro:inertial_box mass="${mass}" x="${sizex}" y="${sizey}" z="${sizez}" />
+	  <xacro:inertial_box mass="${mass}" x="${sizex}" y="${sizey}" z="${sizez}" ox="0.0" oy="0.0" oz="0.0"/>
 	</link>
 	<joint name="${parent}_to_${gps_name}" type="fixed">

Commit message: :+1: implement autonomous function

File: beaverbot_description/urdf/beaverbot.urdf.xacro (robot description, xacro)
@@ -96,5 +96,5 @@
   <xacro:lidar_sensor parent="lidar_base" lidar_name="laser" length="${lidar_length}" radius="${lidar_radius}" mass="${lidar_mass}" ox="0.0" oy="0.0" oz="0.0325" update_rate="${lidar_update_rate}" min_angle="${lidar_min_angle}" max_angle="${lidar_max_angle}" min_range="${lidar_min_range}" max_range="${lidar_max_range}" range_resolution="${lidar_range_resolution}" stdv="${lidar_stdv}" />
   <xacro:imu_sensor parent="back_base_support_frame" imu_name="imu" imu_topic="imu/data_raw" mass="${imu_mass}" sizex="0.03" sizey="0.03" sizez="0.005" ox="0.0" oy="0.0" oz="0.01" update_rate="${imu_update_rate}" noise="${imu_noise}" />
-  <xacro:gps_sensor parent="back_base_support_frame" gps_name="gps" gps_topic="gps/fix" mass="${gps_mass}" sizex="0.03" sizey="0.03" sizez="0.005" ox="0.0" oy="0.0" oz="0.0015" update_rate="${gps_update_rate}" initial_latitude="${gps_latitude}" initial_longitude="${gps_longitude}" noise="${gps_noise}" />
+  <xacro:gps_sensor parent="back_base_support_frame" gps_name="gps" gps_topic="fix" mass="${gps_mass}" sizex="0.03" sizey="0.03" sizez="0.005" ox="0.0" oy="0.0" oz="0.0015" update_rate="${gps_update_rate}" initial_latitude="${gps_latitude}" initial_longitude="${gps_longitude}" noise="${gps_noise}" />
   <xacro:if value="${use_trailer}">
     <xacro:trailer parent="base" trailer_name="trailer" mu1="0.1" mu2="0.1" kp="${kp}" kd="${kd}" />

File: beaverbot_description/urdf/properties.xacro (robot description, xacro)
@@ -45,10 +45,10 @@
   <xacro:property name="imu_update_rate" value="40.0" />
   <xacro:property name="imu_mass" value="0.05" />
-  <xacro:property name="imu_noise" value="0.001" />
+  <xacro:property name="imu_noise" value="0.01" />
   <xacro:property name="gps_update_rate" value="10.0" />
   <xacro:property name="gps_mass" value="0.05" />
-  <xacro:property name="gps_noise" value="0.001" />
-  <xacro:property name="gps_latitude" value="34.835190564394" />
-  <xacro:property name="gps_longitude" value="137.45711512765206" />
+  <xacro:property name="gps_noise" value="0.01" />
+  <xacro:property name="gps_latitude" value="34.70242845166667" />
+  <xacro:property name="gps_longitude" value="137.408935105" />
   <xacro:property name="mu1" value="0.5" />
   <xacro:property name="mu2" value="0.5" />
