Commit message: :+1: update launch files

File: beaverbot_description/urdf/sensors_and_actuators.xacro (robot description, xacro)
@@ -168,4 +168,5 @@
 				<mesh filename="package://beaverbot_description/meshes/cleaner.stl" scale="0.001 0.001 0.001"/>
 			</geometry>
+			<material name="Gray"/>
 			<origin rpy="1.57 0 -1.57" xyz="-0.15 0.4 -0.05" />
 		</visual>
@@ -174,4 +175,5 @@
 				<mesh filename="package://beaverbot_description/meshes/cleaner.stl" scale="0.001 0.001 0.001"/>
 			</geometry>
+			<material name="Gray"/>
 			<origin rpy="1.57 0 -1.57" xyz="-0.15 0.4 -0.05" />
 		</collision>
