Commit message: :+1: update laser scan

File: beaverbot_description/urdf/properties.xacro (robot description, xacro)
@@ -38,5 +38,5 @@
   <xacro:property name="lidar_radius" value="0.0325" />
   <xacro:property name="lidar_min_range" value="0.15" />
-  <xacro:property name="lidar_max_range" value="8.0" />
+  <xacro:property name="lidar_max_range" value="100.0" />
   <xacro:property name="lidar_stdv" value="0.01" />
   <xacro:property name="lidar_range_resolution" value="0.01" />
@@ -55,5 +55,5 @@
   <xacro:property name="kp" value="10000000.0" />
   <xacro:property name="kd" value="1.0" />
-  <xacro:property name="use_trailer" value="true" />
+  <xacro:property name="use_trailer" value="false" />
   <!-- ///////////////////////////////////////////////////////////// -->
 </robot>
